Commit message: configuring joints without controller

File: sanbot_nano_urdf/urdf/sanbot_nano_urdf.urdf (robot description, URDF)
Before this commit: robot sanbot_nano_urdf, 9 links, 8 joints
Links:
- link  body_link: mass 38.598 -> 10.55
- link base_link: mass 12.916 -> 6.0
- link head_link: mass 15.642 -> 2.0
- link neck_link: mass 0.049981 -> 0.014
- link wheel_1_link: mass 0.31873 -> 0.088
- link wheel_2_link: mass 0.31873 -> 0.088
- link wheel_3_link: mass 0.31873 -> 0.088
- link wing_left_link: mass 0.32895 -> 0.091
- link wing_right_link: mass 0.32895 -> 0.091

Commit message: fixing head joints collisions

File: sanbot_nano_urdf/urdf/sanbot_nano_urdf.urdf (robot description, URDF)
Before this commit: robot sanbot_nano_urdf, 9 links, 8 joints
Links:
- link  body_link: mass 10.55 -> 37.769228971116
- link base_link: mass 6.0 -> 12.9158989489561
- link head_link: mass 2.0 -> 15.6411788909065
- link neck_link: mass 0.014 -> 0.077278069019187
- link wheel_1_link: mass 0.088 -> 0.31873
- link wheel_2_link: mass 0.088 -> 0.318731676051724
- link wheel_3_link: mass 0.088 -> 0.318731676051724
- link wing_left_link: mass 0.091 -> 0.328951203332961
- link wing_right_link: mass 0.091 -> 0.328951060786706
Joints:
- joint body: origin xyz=0 0 0.14 rpy=1.5708 0 1.5708 -> xyz=0 0 0.14 rpy=1.5707963267949 0 1.5707963267949
- joint head: limit lower=0 upper=0.646 effort=10 velocity=1 -> lower=0 upper=0.656 effort=10 velocity=1
- joint neck: limit lower=-1.571 upper=1.571 effort=10 velocity=1 -> lower=-1.5708 upper=1.5708 effort=10 velocity=1; origin xyz=0 0.3353 0 rpy=0 0 0 -> xyz=0 0.3344 0 rpy=0 0 0
- joint wheel_2: axis -0.866025403784436 0 -0.500000000000004 -> -0.86603 0 -0.5; origin xyz=-0.0597500000000005 -0.10349003575224 0.03 rpy=1.5707963267949 0 1.5707963267949 -> xyz=-0.05975 -0.10349 0.03 rpy=1.5708 0 1.5708
- joint wheel_3: axis 0.866025403784443 0 -0.499999999999992 -> 0.86603 0 -0.5; origin xyz=-0.0597527016785317 0.103488475937413 0.0299975068501592 rpy=1.5707963267949 0 1.5707963267949 -> xyz=-0.059753 0.10349 0.029998 rpy=1.5708 0 1.5708
- joint wing_left: limit lower=-1.571 upper=3.1416 effort=10 velocity=1 -> lower=-1.5708 upper=3.1416 effort=10 velocity=1
- joint wing_right: limit lower=-1.571 upper=3.1416 effort=10 velocity=1 -> lower=-1.5708 upper=3.1416 effort=10 velocity=1

Commit message: fixing neck joints

File: sanbot_nano_urdf/urdf/sanbot_nano_urdf.urdf (robot description, URDF)
Before this commit: robot sanbot_nano_urdf, 9 links, 8 joints
Links:
- link  body_link: mass 37.769228971116 -> 10.55
- link base_link: mass 12.9158989489561 -> 6.0
- link head_link: mass 15.6411788909065 -> 2.0
- link neck_link: mass 0.077278069019187 -> 0.014
- link wheel_1_link: mass 0.31873 -> 0.088
- link wheel_2_link: mass 0.318731676051724 -> 0.088
- link wheel_3_link: mass 0.318731676051724 -> 0.088
- link wing_left_link: mass 0.328951203332961 -> 0.091
- link wing_right_link: mass 0.328951060786706 -> 0.091
Joints:
- joint neck: origin xyz=0 0.3344 0 rpy=0 0 0 -> xyz=0 0.3444 0 rpy=0 0 0
- joint wheel_1: origin xyz=0.1195 0 0.03 rpy=1.5708 0 1.5708 -> xyz=0.1195 0 0.03 rpy=1.5707963267949 0 1.5707963267949
- joint wheel_2: axis -0.86603 0 -0.5 -> -0.866025403784436 0 -0.500000000000004; origin xyz=-0.05975 -0.10349 0.03 rpy=1.5708 0 1.5708 -> xyz=-0.0597500000000005 -0.10349003575224 0.03 rpy=1.5707963267949 0 1.5707963267949
- joint wheel_3: axis 0.86603 0 -0.5 -> 0.866025403784443 0 -0.499999999999992; origin xyz=-0.059753 0.10349 0.029998 rpy=1.5708 0 1.5708 -> xyz=-0.0597527016785317 0.103488475937413 0.0299975068501592 rpy=1.5707963267949 0 1.5707963267949
- joint wing_right: origin xyz=0.171 0.338 -0.0087685 rpy=0 0 0 -> xyz=0.171 0.337999997444124 -0.00876845650366815 rpy=0 0 0

Commit message: definetelly no head collisions

File: sanbot_nano_urdf/urdf/sanbot_nano_urdf.urdf (robot description, URDF)
Before this commit: robot sanbot_nano_urdf, 9 links, 8 joints
Links:
- link head_link: mass 2.0 -> 2
Joints:
- joint head: axis -1 0 0 -> 1 0 0; origin xyz=0 0.02 0 rpy=0 0 0 -> xyz=0 0.03 0 rpy=0 0 0
- joint neck: origin xyz=0 0.3444 0 rpy=0 0 0 -> xyz=0 0.3344 0 rpy=0 0 0
- joint wing_left: origin xyz=-0.171 0.338 -0.0087685 rpy=0 0 0 -> xyz=-0.171 0.337999997444124 -0.00876845650366815 rpy=0 0 0
- joint wing_right: origin xyz=0.171 0.337999997444124 -0.00876845650366815 rpy=0 0 0 -> xyz=0.171 0.338 -0.0087685 rpy=0 0 0

Commit message: wings and head joints control ok, still have to work on solid to max limits for head

File: sanbot_nano_urdf/urdf/sanbot_nano_urdf.urdf (robot description, URDF)
Before this commit: robot sanbot_nano_urdf, 9 links, 8 joints
Links:
- link head_link: mass 2 -> 0.5
Joints:
- joint head: limit lower=0 upper=0.656 effort=10 velocity=1 -> lower=0 upper=0.656 effort=2 velocity=0.5
- joint neck: limit lower=-1.5708 upper=1.5708 effort=10 velocity=1 -> lower=-1.5708 upper=1.5708 effort=2 velocity=0.5
- joint wing_right: axis -1 0 0 -> 1 0 0

Commit message: trying head tilt centered in the head

File: sanbot_nano_urdf/urdf/sanbot_nano_urdf.urdf (robot description, URDF)
Before this commit: robot sanbot_nano_urdf, 9 links, 8 joints
Joints:
- joint head: axis 1 0 0 -> 0 1 0; limit lower=0 upper=0.656 effort=2 velocity=0.5 -> lower=0 upper=0.656 effort=2 velocity=1; origin xyz=0 0.03 0 rpy=0 0 0 -> xyz=0.245 0 0 rpy=0 0 0
- joint neck: axis 0 -1 0 -> -1 0 0; limit lower=-1.5708 upper=1.5708 effort=2 velocity=0.5 -> lower=-1.5708 upper=1.5708 effort=2 velocity=1; origin xyz=0 0.3344 0 rpy=0 0 0 -> xyz=0 0.3074 0 rpy=0 0 1.5708
- joint wing_left: origin xyz=-0.171 0.337999997444124 -0.00876845650366815 rpy=0 0 0 -> xyz=-0.171 0.338 -0.0087685 rpy=0 0 0

Commit message: all joints full movement and final adjustment of weights

File: sanbot_nano_urdf/urdf/sanbot_nano_urdf.urdf (robot description, URDF)
Before this commit: robot sanbot_nano_urdf, 9 links, 8 joints
Links:
- link  body_link: mass 10.55 -> 10.54
- link head_link: mass 0.5 -> 2.0
Joints:
- joint head: axis 0 1 0 -> 0 -1 0

Commit message: adding joints for camera and giroscope

File: sanbot_nano_urdf/urdf/sanbot_nano_urdf.urdf (robot description, URDF)
Before this commit: robot sanbot_nano_urdf, 9 links, 8 joints
Links:
- added link camera_chin_Link, mass 0.001; collision mesh filename=package://sanbot_nano_urdf/meshes/camera_chin_Link.STL; visual mesh filename=package://sanbot_nano_urdf/meshes/camera_chin_Link.STL
- added link giroscope_link, mass 0.001; collision mesh filename=package://sanbot_nano_urdf/meshes/giroscope_link.STL; visual mesh filename=package://sanbot_nano_urdf/meshes/giroscope_link.STL
- link wing_left_link: mass 0.091 -> 0.09
- link wing_right_link: mass 0.091 -> 0.09
Joints:
- added joint camera_chin: type fixed, parent head_link, child camera_chin_Link, origin xyz=-0.0570293736770144 0 -0.143348462664648 rpy=0 0 -1.5707963267949, axis 0 0 0
- added joint giroscope: type fixed, parent base_link, child giroscope_link, origin xyz=0 0 0.13 rpy=1.5708 0 1.5708, axis 0 0 0
- joint neck: origin xyz=0 0.3074 0 rpy=0 0 1.5708 -> xyz=0 0.3074 0 rpy=0 0 1.5707963267949
- joint wing_left: origin xyz=-0.171 0.338 -0.0087685 rpy=0 0 0 -> xyz=-0.171 0.337999997444124 -0.00876845650366815 rpy=0 0 0
- joint wing_right: origin xyz=0.171 0.338 -0.0087685 rpy=0 0 0 -> xyz=0.171 0.337999997444124 -0.00876845650366815 rpy=0 0 0

Commit message: camera out and not ir

File: sanbot_nano_urdf/urdf/sanbot_nano_urdf.urdf (robot description, URDF)
Before this commit: robot sanbot_nano_urdf, 11 links, 10 joints
Joints:
- joint camera_chin: axis 0 0 0 -> 0 0 1; origin xyz=-0.0570293736770144 0 -0.143348462664648 rpy=0 0 -1.5707963267949 -> xyz=-0.08 0 -0.1355 rpy=0 0 -1.5708

Commit message: closing chest and adjusting robot size

File: sanbot_nano_urdf/urdf/sanbot_nano_urdf.urdf (robot description, URDF)
Before this commit: robot sanbot_nano_urdf, 11 links, 10 joints
Joints:
- joint body: origin xyz=0 0 0.14 rpy=1.5707963267949 0 1.5707963267949 -> xyz=0 0 0.14 rpy=1.5708 0 1.5708
- joint camera_chin: axis 0 0 1 -> 0 0 0
- joint head: origin xyz=0.245 0 0 rpy=0 0 0 -> xyz=0 0.165 0 rpy=0 0 1.5708
- joint neck: axis -1 0 0 -> 0 -1 0; origin xyz=0 0.3074 0 rpy=0 0 1.5707963267949 -> xyz=0 0.37832 0 rpy=0 0 0
- joint wing_left: origin xyz=-0.171 0.337999997444124 -0.00876845650366815 rpy=0 0 0 -> xyz=-0.171 0.338 -0.0087685 rpy=0 0 0
- joint wing_right: origin xyz=0.171 0.337999997444124 -0.00876845650366815 rpy=0 0 0 -> xyz=0.171 0.338 -0.0087685 rpy=0 0 0

Commit message: camera transmiting and simple README with features

File: sanbot_nano_urdf/urdf/sanbot_nano_urdf.urdf (robot description, URDF)
Before this commit: robot sanbot_nano_urdf, 11 links, 10 joints
Links:
- removed link camera_chin_Link
- added link camera_chin_link, mass 0.001; collision mesh filename=package://sanbot_nano_urdf/meshes/camera_chin_link.STL; visual mesh filename=package://sanbot_nano_urdf/meshes/camera_chin_link.STL
Joints:
- joint camera_chin: child camera_chin_Link -> camera_chin_link

Commit message: new urdf after aesthetic and gyro removal

File: sanbot_nano_urdf/urdf/sanbot_nano_urdf.urdf (robot description, URDF)
Before this commit: robot sanbot_nano_urdf, 11 links, 10 joints
Links:
- removed link giroscope_link
- link camera_chin_link: mass 0.001 -> 0.002
Joints:
- removed joint giroscope
- joint body: origin xyz=0 0 0.14 rpy=1.5708 0 1.5708 -> xyz=0 0 0.14 rpy=1.5707963267949 0 1.5707963267949
- joint camera_chin: child camera_chin_link -> camera_chin_Link
- joint wing_left: origin xyz=-0.171 0.338 -0.0087685 rpy=0 0 0 -> xyz=-0.171 0.337999997444124 -0.00876845650366815 rpy=0 0 0
- joint wing_right: origin xyz=0.171 0.338 -0.0087685 rpy=0 0 0 -> xyz=0.171 0.337999997444124 -0.00876845650366815 rpy=0 0 0

Commit message: adding velocity controllers for wheels and adjusting other plugins

File: sanbot_nano_urdf/urdf/sanbot_nano_urdf.urdf (robot description, URDF)
Before this commit: robot sanbot_nano_urdf, 10 links, 9 joints
Links:
- removed link wheel_1_link
- removed link wheel_2_link
- removed link wheel_3_link
- added link wheel_back_link, mass 0.088; collision mesh filename=package://sanbot_nano_urdf/meshes/wheel_back_link.STL; visual mesh filename=package://sanbot_nano_urdf/meshes/wheel_back_link.STL
- added link wheel_left_link, mass 0.088; collision mesh filename=package://sanbot_nano_urdf/meshes/wheel_left_link.STL; visual mesh filename=package://sanbot_nano_urdf/meshes/wheel_left_link.STL
- added link wheel_right_link, mass 0.088; collision mesh filename=package://sanbot_nano_urdf/meshes/wheel_right_link.STL; visual mesh filename=package://sanbot_nano_urdf/meshes/wheel_right_link.STL
Joints:
- removed joint wheel_1
- removed joint wheel_2
- removed joint wheel_3
- added joint wheel_back: type continuous, parent base_link, child wheel_back_link, origin xyz=0.1195 0 0.03 rpy=1.5707963267949 0 1.5707963267949, axis 0 0 1
- added joint wheel_left: type continuous, parent base_link, child wheel_left_link, origin xyz=-0.0597500000000005 -0.10349003575224 0.03 rpy=1.5707963267949 0 1.5707963267949, axis -0.866025403784436 0 -0.500000000000004
- added joint wheel_right: type continuous, parent base_link, child wheel_right_link, origin xyz=-0.0597527016785317 0.103488475937413 0.0299975068501592 rpy=1.5707963267949 0 1.5707963267949, axis 0.866025403784443 0 -0.499999999999992
- joint camera_chin: child camera_chin_Link -> camera_chin_link

Commit message: adding collada files to give color to model

File: sanbot_nano_urdf/urdf/sanbot_nano_urdf.urdf (robot description, URDF)
Before this commit: robot sanbot_nano_urdf, 10 links, 9 joints
Links:
- link  body_link: geometry collision mesh filename=package://sanbot_nano_urdf/meshes/body_link.STL; visual mesh filename=package://sanbot_nano_urdf/textures/body.dae scale=1 1 1
- link base_link: geometry collision mesh filename=package://sanbot_nano_urdf/meshes/base_link.STL; visual mesh filename=package://sanbot_nano_urdf/textures/base.dae scale=1 1 1
- link camera_chin_link: geometry collision mesh filename=package://sanbot_nano_urdf/meshes/camera_chin_link.STL; visual mesh filename=package://sanbot_nano_urdf/textures/camera_chin.dae scale=1 1 1
- link head_link: geometry collision mesh filename=package://sanbot_nano_urdf/meshes/head_link.STL; visual mesh filename=package://sanbot_nano_urdf/textures/head.dae scale=1 1 1
- link neck_link: geometry collision mesh filename=package://sanbot_nano_urdf/meshes/neck_link.STL; visual mesh filename=package://sanbot_nano_urdf/textures/neck.dae scale=1 1 1
- link wing_left_link: geometry collision mesh filename=package://sanbot_nano_urdf/meshes/wing_left_link.STL; visual mesh filename=package://sanbot_nano_urdf/textures/wing_left.dae scale=1 1 1
- link wing_right_link: geometry collision mesh filename=package://sanbot_nano_urdf/meshes/wing_right_link.STL; visual mesh filename=package://sanbot_nano_urdf/textures/wing_right.dae scale=1 1 1

Commit message: adjusting global origin and removing odometry topc

File: sanbot_nano_urdf/urdf/sanbot_nano_urdf.urdf (robot description, URDF)
Before this commit: robot sanbot_nano_urdf, 10 links, 9 joints
Links:
- removed link  body_link
- added link body_link, mass 10.54; collision mesh filename=package://sanbot_nano_urdf/meshes/body_link.STL; visual mesh filename=package://sanbot_nano_urdf/meshes/body_link.STL
- link base_link: geometry collision mesh filename=package://sanbot_nano_urdf/meshes/base_link.STL; visual mesh filename=package://sanbot_nano_urdf/meshes/base_link.STL
- link camera_chin_link: geometry collision mesh filename=package://sanbot_nano_urdf/meshes/camera_chin_link.STL; visual mesh filename=package://sanbot_nano_urdf/meshes/camera_chin_link.STL
- link head_link: geometry collision mesh filename=package://sanbot_nano_urdf/meshes/head_link.STL; visual mesh filename=package://sanbot_nano_urdf/meshes/head_link.STL
- link neck_link: geometry collision mesh filename=package://sanbot_nano_urdf/meshes/neck_link.STL; visual mesh filename=package://sanbot_nano_urdf/meshes/neck_link.STL
- link wing_left_link: geometry collision mesh filename=package://sanbot_nano_urdf/meshes/wing_left_link.STL; visual mesh filename=package://sanbot_nano_urdf/meshes/wing_left_link.STL
- link wing_right_link: geometry collision mesh filename=package://sanbot_nano_urdf/meshes/wing_right_link.STL; visual mesh filename=package://sanbot_nano_urdf/meshes/wing_right_link.STL
Joints:
- joint body: child  body_link -> body_link; origin xyz=0 0 0.14 rpy=1.5707963267949 0 1.5707963267949 -> xyz=0 0 0.14 rpy=1.5707963267949 0 -1.5707963267949
- joint camera_chin: origin xyz=-0.08 0 -0.1355 rpy=0 0 -1.5708 -> xyz=-0.0799999999999998 0 -0.1355 rpy=0 0 -1.5707963267949
- joint head: origin xyz=0 0.165 0 rpy=0 0 1.5708 -> xyz=0 0.165 0 rpy=0 0 1.5707963267949
- joint neck: origin xyz=0 0.37832 0 rpy=0 0 0 -> xyz=0 0.37832467677926 0 rpy=0 0 0; parent  body_link -> body_link
- joint wheel_back: origin xyz=0.1195 0 0.03 rpy=1.5707963267949 0 1.5707963267949 -> xyz=-0.1195 0 0.03 rpy=1.5707963267949 0 -1.5707963267949
- joint wheel_left: origin xyz=-0.0597500000000005 -0.10349003575224 0.03 rpy=1.5707963267949 0 1.5707963267949 -> xyz=0.0597500000000005 0.10349003575224 0.03 rpy=1.5707963267949 0 -1.5707963267949
- joint wheel_right: origin xyz=-0.0597527016785317 0.103488475937413 0.0299975068501592 rpy=1.5707963267949 0 1.5707963267949 -> xyz=0.0597527016785317 -0.103488475937413 0.0299975068501592 rpy=1.5707963267949 0 -1.5707963267949
- joint wing_left: parent  body_link -> body_link
- joint wing_right: parent  body_link -> body_link

Commit message: adding forehead and depth camera to solid and urdf files

File: sanbot_nano_urdf/urdf/sanbot_nano_urdf.urdf (robot description, URDF)
Before this commit: robot sanbot_nano_urdf, 10 links, 9 joints
Links:
- added link camera_depth_link, mass 0.0024849; collision mesh filename=package://sanbot_nano_urdf/meshes/camera_depth_link.STL; visual mesh filename=package://sanbot_nano_urdf/meshes/camera_depth_link.STL
- added link camera_forehead_link, mass 0.00068843; collision mesh filename=package://sanbot_nano_urdf/meshes/camera_forehead_link.STL; visual mesh filename=package://sanbot_nano_urdf/meshes/camera_forehead_link.STL
Joints:
- added joint camera_depth: type fixed, parent head_link, child camera_depth_link, origin xyz=0.106924212815129 0 -0.13500000000001 rpy=-3.14159265358979 0 1.5707963267949, axis 0 0 0
- added joint camera_forehead: type fixed, parent head_link, child camera_forehead_link, origin xyz=0.101924212815131 -0.0850000000000006 -0.136000000000001 rpy=-3.14159265358979 0 1.5707963267949, axis 0 0 0

Commit message: adding cameras plugin and many small adjustments

File: sanbot_nano_urdf/urdf/sanbot_nano_urdf.urdf (robot description, URDF)
Before this commit: robot sanbot_nano_urdf, 12 links, 11 joints
Joints:
- removed joint head
- removed joint neck
- added joint head_pan: type revolute, parent body_link, child neck_link, origin xyz=0 0.37832467677926 0 rpy=0 0 0, axis 0 -1 0, limit lower=-1.5708 upper=1.5708 effort=2 velocity=1
- added joint head_tilt: type revolute, parent neck_link, child head_link, origin xyz=0 0.165 0 rpy=0 0 1.5707963267949, axis 0 -1 0, limit lower=0 upper=0.656 effort=2 velocity=1

Commit message: adding collada to urdf

File: sanbot_nano_urdf/urdf/sanbot_nano_urdf.urdf (robot description, URDF)
Before this commit: robot sanbot_nano_urdf, 12 links, 11 joints
Links:
- link base_link: geometry collision mesh filename=package://sanbot_nano_urdf/meshes/base_link.STL; visual mesh filename=package://sanbot_nano_urdf/textures/base.dae
- link body_link: geometry collision mesh filename=package://sanbot_nano_urdf/meshes/body_link.STL; visual mesh filename=package://sanbot_nano_urdf/textures/body.dae
- link camera_chin_link: geometry collision mesh filename=package://sanbot_nano_urdf/meshes/camera_chin_link.STL; visual mesh filename=package://sanbot_nano_urdf/textures/camera_chin.dae
- link camera_depth_link: geometry collision mesh filename=package://sanbot_nano_urdf/meshes/camera_depth_link.STL; visual mesh filename=package://sanbot_nano_urdf/textures/camera_depth.dae
- link camera_forehead_link: geometry collision mesh filename=package://sanbot_nano_urdf/meshes/camera_forehead_link.STL; visual mesh filename=package://sanbot_nano_urdf/textures/camera_forehead.dae
- link head_link: geometry collision mesh filename=package://sanbot_nano_urdf/meshes/head_link.STL; visual mesh filename=package://sanbot_nano_urdf/textures/head.dae
- link wing_left_link: geometry collision mesh filename=package://sanbot_nano_urdf/meshes/wing_left_link.STL; visual mesh filename=package://sanbot_nano_urdf/textures/wing_left.dae
- link wing_right_link: geometry collision mesh filename=package://sanbot_nano_urdf/meshes/wing_right_link.STL; visual mesh filename=package://sanbot_nano_urdf/textures/wing_right.dae

Commit message: testing 1 ir sensor

File: sanbot_nano_urdf/urdf/sanbot_nano_urdf.urdf (robot description, URDF)
Before this commit: robot sanbot_nano_urdf, 12 links, 11 joints
Links:
- added link ir_13_link, mass 0.001; collision mesh filename=package://sanbot_nano_urdf/meshes/ir_13_link.STL; visual mesh filename=package://sanbot_nano_urdf/meshes/ir_13_link.STL
- link base_link: geometry collision mesh filename=package://sanbot_nano_urdf/meshes/base_link.STL; visual mesh filename=package://sanbot_nano_urdf/meshes/base_link.STL
- link body_link: geometry collision mesh filename=package://sanbot_nano_urdf/meshes/body_link.STL; visual mesh filename=package://sanbot_nano_urdf/meshes/body_link.STL
- link camera_chin_link: mass 0.002 -> 8.42614806857185E-05; geometry collision mesh filename=package://sanbot_nano_urdf/meshes/camera_chin_link.STL; visual mesh filename=package://sanbot_nano_urdf/meshes/camera_chin_link.STL
- link camera_depth_link: geometry collision mesh filename=package://sanbot_nano_urdf/meshes/camera_depth_link.STL; visual mesh filename=package://sanbot_nano_urdf/meshes/camera_depth_link.STL
- link camera_forehead_link: geometry collision mesh filename=package://sanbot_nano_urdf/meshes/camera_forehead_link.STL; visual mesh filename=package://sanbot_nano_urdf/meshes/camera_forehead_link.STL
- link head_link: geometry collision mesh filename=package://sanbot_nano_urdf/meshes/head_link.STL; visual mesh filename=package://sanbot_nano_urdf/meshes/head_link.STL
- link wing_left_link: geometry collision mesh filename=package://sanbot_nano_urdf/meshes/wing_left_link.STL; visual mesh filename=package://sanbot_nano_urdf/meshes/wing_left_link.STL
- link wing_right_link: geometry collision mesh filename=package://sanbot_nano_urdf/meshes/wing_right_link.STL; visual mesh filename=package://sanbot_nano_urdf/meshes/wing_right_link.STL
Joints:
- added joint ir_13: type fixed, parent body_link, child ir_13_link, origin xyz=0 0.23 -0.16 rpy=0 0 0, axis 0 0 0
- joint camera_depth: origin xyz=0.106924212815129 0 -0.13500000000001 rpy=-3.14159265358979 0 1.5707963267949 -> xyz=0.10692 0 -0.135 rpy=-3.1416 0 1.5708
- joint camera_forehead: origin xyz=0.101924212815131 -0.0850000000000006 -0.136000000000001 rpy=-3.14159265358979 0 1.5707963267949 -> xyz=0.10192 -0.085 -0.136 rpy=-3.1416 0 1.5708
- joint wing_left: origin xyz=-0.171 0.337999997444124 -0.00876845650366815 rpy=0 0 0 -> xyz=-0.171 0.338 -0.0087685 rpy=0 0 0
- joint wing_right: origin xyz=0.171 0.337999997444124 -0.00876845650366815 rpy=0 0 0 -> xyz=0.171 0.338 -0.0087685 rpy=0 0 0
