Commit message: adding ir sensors to solid and urdf files

File: sanbot_nano_urdf/urdf/sanbot_nano_urdf.urdf (robot description, URDF)
Before this commit: robot sanbot_nano_urdf, 12 links, 11 joints
Links:
- added link ir_10_link, mass 0.001; collision mesh filename=package://sanbot_nano_urdf/meshes/ir_10_link.STL; visual mesh filename=package://sanbot_nano_urdf/meshes/ir_10_link.STL
- added link ir_11_link, mass 0.001; collision mesh filename=package://sanbot_nano_urdf/meshes/ir_11_link.STL; visual mesh filename=package://sanbot_nano_urdf/meshes/ir_11_link.STL
- added link ir_12_link, mass 0.001; collision mesh filename=package://sanbot_nano_urdf/meshes/ir_12_link.STL; visual mesh filename=package://sanbot_nano_urdf/meshes/ir_12_link.STL
- added link ir_13_link, mass 0.001; collision mesh filename=package://sanbot_nano_urdf/meshes/ir_13_link.STL; visual mesh filename=package://sanbot_nano_urdf/meshes/ir_13_link.STL
- added link ir_14_link, mass 0.001; collision mesh filename=package://sanbot_nano_urdf/meshes/ir_14_link.STL; visual mesh filename=package://sanbot_nano_urdf/meshes/ir_14_link.STL
- added link ir_15_link, mass 0.001; collision mesh filename=package://sanbot_nano_urdf/meshes/ir_15_link.STL; visual mesh filename=package://sanbot_nano_urdf/meshes/ir_15_link.STL
- added link ir_16_link, mass 0.001; collision mesh filename=package://sanbot_nano_urdf/meshes/ir_16_link.STL; visual mesh filename=package://sanbot_nano_urdf/meshes/ir_16_link.STL
- added link ir_17_link, mass 0.001; collision mesh filename=package://sanbot_nano_urdf/meshes/ir_17_link.STL; visual mesh filename=package://sanbot_nano_urdf/meshes/ir_17_link.STL
- added link ir_1_link, mass 0.001; collision mesh filename=package://sanbot_nano_urdf/meshes/ir_1_link.STL; visual mesh filename=package://sanbot_nano_urdf/meshes/ir_1_link.STL
- added link ir_2_link, mass 0.001; collision mesh filename=package://sanbot_nano_urdf/meshes/ir_2_link.STL; visual mesh filename=package://sanbot_nano_urdf/meshes/ir_2_link.STL
- added link ir_3_link, mass 0.001; collision mesh filename=package://sanbot_nano_urdf/meshes/ir_3_link.STL; visual mesh filename=package://sanbot_nano_urdf/meshes/ir_3_link.STL
- added link ir_4_link, mass 0.001; collision mesh filename=package://sanbot_nano_urdf/meshes/ir_4_link.STL; visual mesh filename=package://sanbot_nano_urdf/meshes/ir_4_link.STL
- added link ir_5_link, mass 0.001; collision mesh filename=package://sanbot_nano_urdf/meshes/ir_5_link.STL; visual mesh filename=package://sanbot_nano_urdf/meshes/ir_5_link.STL
- added link ir_6_link, mass 0.001; collision mesh filename=package://sanbot_nano_urdf/meshes/ir_6_link.STL; visual mesh filename=package://sanbot_nano_urdf/meshes/ir_6_link.STL
- added link ir_7_Link, mass 0.001; collision mesh filename=package://sanbot_nano_urdf/meshes/ir_7_Link.STL; visual mesh filename=package://sanbot_nano_urdf/meshes/ir_7_Link.STL
- added link ir_8_Link, mass 0.001; collision mesh filename=package://sanbot_nano_urdf/meshes/ir_8_Link.STL; visual mesh filename=package://sanbot_nano_urdf/meshes/ir_8_Link.STL
- added link ir_9_link, mass 0.001; collision mesh filename=package://sanbot_nano_urdf/meshes/ir_9_link.STL; visual mesh filename=package://sanbot_nano_urdf/meshes/ir_9_link.STL
- link base_link: geometry collision mesh filename=package://sanbot_nano_urdf/meshes/base_link.STL; visual mesh filename=package://sanbot_nano_urdf/meshes/base_link.STL
- link body_link: geometry collision mesh filename=package://sanbot_nano_urdf/meshes/body_link.STL; visual mesh filename=package://sanbot_nano_urdf/meshes/body_link.STL
- link camera_chin_link: mass 0.002 -> 8.4261E-05; geometry collision mesh filename=package://sanbot_nano_urdf/meshes/camera_chin_link.STL; visual mesh filename=package://sanbot_nano_urdf/meshes/camera_chin_link.STL
- link camera_depth_link: geometry collision mesh filename=package://sanbot_nano_urdf/meshes/camera_depth_link.STL; visual mesh filename=package://sanbot_nano_urdf/meshes/camera_depth_link.STL
- link camera_forehead_link: geometry collision mesh filename=package://sanbot_nano_urdf/meshes/camera_forehead_link.STL; visual mesh filename=package://sanbot_nano_urdf/meshes/camera_forehead_link.STL
- link head_link: geometry collision mesh filename=package://sanbot_nano_urdf/meshes/head_link.STL; visual mesh filename=package://sanbot_nano_urdf/meshes/head_link.STL
- link wing_left_link: geometry collision mesh filename=package://sanbot_nano_urdf/meshes/wing_left_link.STL; visual mesh filename=package://sanbot_nano_urdf/meshes/wing_left_link.STL
- link wing_right_link: geometry collision mesh filename=package://sanbot_nano_urdf/meshes/wing_right_link.STL; visual mesh filename=package://sanbot_nano_urdf/meshes/wing_right_link.STL
Joints:
- added joint ir_1: type fixed, parent base_link, child ir_1_link, origin xyz=0.14595 0.084263 0.015 rpy=1.3735 0.11271 -1.0584, axis 0 0 0
- added joint ir_10: type fixed, parent base_link, child ir_10_link, origin xyz=0.055169 -0.16979 0.0775 rpy=1.5708 0 2.0595, axis 0 0 0
- added joint ir_11: type fixed, parent body_link, child ir_11_link, origin xyz=0.029354 0.08 -0.15843 rpy=0 0 0, axis 0 0 0
- added joint ir_12: type fixed, parent body_link, child ir_12_link, origin xyz=-0.030733 0.08 -0.15817 rpy=0 0 0, axis 0 0 0
- added joint ir_13: type fixed, parent body_link, child ir_13_link, origin xyz=0 0.23 -0.16 rpy=0 0 0, axis 0 0 0
- added joint ir_14: type fixed, parent wing_right_link, child ir_14_link, origin xyz=0.0185 0.017 -0.045 rpy=0.5236 0 0, axis 0 0 0
- added joint ir_15: type fixed, parent wing_right_link, child ir_15_link, origin xyz=0.0185 -0.15329 -0.045 rpy=-0.34907 0 0, axis 0 0 0
- added joint ir_16: type fixed, parent wing_left_link, child ir_16_link, origin xyz=-0.0185 0.017 -0.045 rpy=0.5236 0 0, axis 0 0 0
- added joint ir_17: type fixed, parent wing_left_link, child ir_17_link, origin xyz=-0.0185 -0.15329 -0.045 rpy=-0.34907 0 0, axis 0 0 0
- added joint ir_2: type fixed, parent base_link, child ir_2_link, origin xyz=0.14595 -0.084263 0.015 rpy=1.3735 -0.11271 -2.0832, axis 0 0 0
- added joint ir_3: type fixed, parent base_link, child ir_3_link, origin xyz=0.055169 0.16979 0.0775 rpy=1.5708 0 -1.885, axis 0 0 0
- added joint ir_4: type fixed, parent base_link, child ir_4_link, origin xyz=0.10493 0.14443 0.0775 rpy=1.5708 0 -2.1991, axis 0 0 0
- added joint ir_5: type fixed, parent base_link, child ir_5_link, origin xyz=0.14443 0.10493 0.0775 rpy=1.5708 0 -2.5133, axis 0 0 0
- added joint ir_6: type fixed, parent base_link, child ir_6_link, origin xyz=0.16979 0.055169 0.0775 rpy=1.5708 0 -2.8274, axis 0 0 0
- added joint ir_7: type fixed, parent base_link, child ir_7_Link, origin xyz=0.16979 -0.055169 0.0775 rpy=1.5708 0 2.8274, axis 0 0 0
- added joint ir_8: type fixed, parent base_link, child ir_8_Link, origin xyz=0.14443 -0.10493 0.0775 rpy=1.5708 0 2.5133, axis 0 0 0
- added joint ir_9: type fixed, parent base_link, child ir_9_link, origin xyz=0.10493 -0.14443 0.0775 rpy=1.5708 0 2.3736, axis 0 0 0
- joint body: origin xyz=0 0 0.14 rpy=1.5707963267949 0 -1.5707963267949 -> xyz=0 0 0.14 rpy=1.5708 0 -1.5708
- joint camera_chin: origin xyz=-0.0799999999999998 0 -0.1355 rpy=0 0 -1.5707963267949 -> xyz=-0.08 0 -0.1355 rpy=0 0 -1.5708
- joint camera_depth: origin xyz=0.106924212815129 0 -0.13500000000001 rpy=-3.14159265358979 0 1.5707963267949 -> xyz=0.10692 0 -0.135 rpy=-3.1416 0 1.5708
- joint camera_forehead: origin xyz=0.101924212815131 -0.0850000000000006 -0.136000000000001 rpy=-3.14159265358979 0 1.5707963267949 -> xyz=0.10192 -0.085 -0.136 rpy=-3.1416 0 1.5708
- joint head_pan: origin xyz=0 0.37832467677926 0 rpy=0 0 0 -> xyz=0 0.37832 0 rpy=0 0 0
- joint head_tilt: origin xyz=0 0.165 0 rpy=0 0 1.5707963267949 -> xyz=0 0.165 0 rpy=0 0 1.5708
- joint wheel_back: origin xyz=-0.1195 0 0.03 rpy=1.5707963267949 0 -1.5707963267949 -> xyz=-0.1195 0 0.03 rpy=1.5708 0 -1.5708
- joint wheel_left: axis -0.866025403784436 0 -0.500000000000004 -> -0.86603 0 -0.5; origin xyz=0.0597500000000005 0.10349003575224 0.03 rpy=1.5707963267949 0 -1.5707963267949 -> xyz=0.05975 0.10349 0.03 rpy=1.5708 0 -1.5708
- joint wheel_right: axis 0.866025403784443 0 -0.499999999999992 -> 0.86603 0 -0.5; origin xyz=0.0597527016785317 -0.103488475937413 0.0299975068501592 rpy=1.5707963267949 0 -1.5707963267949 -> xyz=0.059753 -0.10349 0.029998 rpy=1.5708 0 -1.5708
- joint wing_left: origin xyz=-0.171 0.337999997444124 -0.00876845650366815 rpy=0 0 0 -> xyz=-0.171 0.338 -0.0087685 rpy=0 0 0
- joint wing_right: origin xyz=0.171 0.337999997444124 -0.00876845650366815 rpy=0 0 0 -> xyz=0.171 0.338 -0.0087685 rpy=0 0 0

Commit message: adding ir plugins on urdf

File: sanbot_nano_urdf/urdf/sanbot_nano_urdf.urdf (robot description, URDF)
Before this commit: robot sanbot_nano_urdf, 29 links, 28 joints
Links:
- removed link ir_7_Link
- removed link ir_8_Link
- added link ir_7_link, mass 0.001; collision mesh filename=package://sanbot_nano_urdf/meshes/ir_7_link.STL; visual mesh filename=package://sanbot_nano_urdf/meshes/ir_7_link.STL
- added link ir_8_link, mass 0.001; collision mesh filename=package://sanbot_nano_urdf/meshes/ir_8_link.STL; visual mesh filename=package://sanbot_nano_urdf/meshes/ir_8_link.STL
Joints:
- joint ir_7: child ir_7_Link -> ir_7_link
- joint ir_8: child ir_8_Link -> ir_8_link

Commit message: final changes to ir and adding textures

File: sanbot_nano_urdf/urdf/sanbot_nano_urdf.urdf (robot description, URDF)
Before this commit: robot sanbot_nano_urdf, 29 links, 28 joints
Joints:
- joint body: origin xyz=0 0 0.14 rpy=1.5708 0 -1.5708 -> xyz=0 0 0.14 rpy=1.5707963267949 0 -1.5707963267949
- joint camera_chin: origin xyz=-0.08 0 -0.1355 rpy=0 0 -1.5708 -> xyz=-0.0799999999999998 0 -0.1355 rpy=0 0 -1.5707963267949
- joint camera_depth: origin xyz=0.10692 0 -0.135 rpy=-3.1416 0 1.5708 -> xyz=0.106924212815129 0 -0.135000000000008 rpy=-3.14159265358979 0 1.5707963267949
- joint camera_forehead: origin xyz=0.10192 -0.085 -0.136 rpy=-3.1416 0 1.5708 -> xyz=0.101924212815131 -0.085 -0.136 rpy=-3.14159265358979 0 1.5707963267949
- joint head_pan: origin xyz=0 0.37832 0 rpy=0 0 0 -> xyz=0 0.37832467677926 0 rpy=0 0 0
- joint head_tilt: origin xyz=0 0.165 0 rpy=0 0 1.5708 -> xyz=0 0.165 0 rpy=0 0 1.5707963267949
- joint ir_1: origin xyz=0.14595 0.084263 0.015 rpy=1.3735 0.11271 -1.0584 -> xyz=0.145947826146462 0.0842630167133011 0.015 rpy=1.38875485932488 0.104144000510505 -1.05671160838547
- joint ir_10: origin xyz=0.055169 -0.16979 0.0775 rpy=1.5708 0 2.0595 -> xyz=0.0348282680125839 -0.17509352722209 0.0775 rpy=1.5707963267949 0 1.76714586764425
- joint ir_11: origin xyz=0.029354 0.08 -0.15843 rpy=0 0 0 -> xyz=0.0293538954235705 0.08 -0.158431357507698 rpy=0 0 0
- joint ir_12: origin xyz=-0.030733 0.08 -0.15817 rpy=0 0 0 -> xyz=-0.0307326300261287 0.08 -0.158169692640364 rpy=0 0 0
- joint ir_14: origin xyz=0.0185 0.017 -0.045 rpy=0.5236 0 0 -> xyz=0.0185 0.0219999970218235 -0.045 rpy=0.78539816339745 0 0
- joint ir_15: origin xyz=0.0185 -0.15329 -0.045 rpy=-0.34907 0 0 -> xyz=0.0185 -0.123285030574576 -0.045 rpy=0 0 0
- joint ir_16: origin xyz=-0.0185 0.017 -0.045 rpy=0.5236 0 0 -> xyz=-0.0185000000000005 0.0219999970208385 -0.0450000000004853 rpy=0.78539816339745 0 0
- joint ir_17: origin xyz=-0.0185 -0.15329 -0.045 rpy=-0.34907 0 0 -> xyz=-0.0184999999999998 -0.123285030575561 -0.0449999999973061 rpy=0 0 0
- joint ir_2: origin xyz=0.14595 -0.084263 0.015 rpy=1.3735 -0.11271 -2.0832 -> xyz=0.145947826146462 -0.0842630167133002 0.015 rpy=1.38875485932488 -0.104144000510505 -2.08488104520432
- joint ir_3: origin xyz=0.055169 0.16979 0.0775 rpy=1.5708 0 -1.885 -> xyz=0.034828268012584 0.17509352722209 0.0775 rpy=1.5707963267949 0 -1.76714586764426
- joint ir_4: origin xyz=0.10493 0.14443 0.0775 rpy=1.5708 0 -2.1991 -> xyz=0.0991824752043695 0.148437063946314 0.0775 rpy=1.5707963267949 0 -2.15984494934298
- joint ir_5: origin xyz=0.14443 0.10493 0.0775 rpy=1.5708 0 -2.5133 -> xyz=0.148436951264281 0.0991823999126595 0.0775 rpy=1.5707963267949 0 -2.55254403104171
- joint ir_6: origin xyz=0.16979 0.055169 0.0775 rpy=1.5708 0 -2.8274 -> xyz=0.175093148705453 0.0348281927209758 0.0775 rpy=1.5707963267949 0 -2.94524311274043
- joint ir_7: origin xyz=0.16979 -0.055169 0.0775 rpy=1.5708 0 2.8274 -> xyz=0.175093148705452 -0.0348281927209761 0.0775 rpy=1.5707963267949 0 2.94524311274043
- joint ir_8: origin xyz=0.14443 -0.10493 0.0775 rpy=1.5708 0 2.5133 -> xyz=0.148436951264281 -0.0991823999126594 0.0775 rpy=1.5707963267949 0 2.5525440310417
- joint ir_9: origin xyz=0.10493 -0.14443 0.0775 rpy=1.5708 0 2.3736 -> xyz=0.0991824752043694 -0.148437063946314 0.0775 rpy=1.5707963267949 0 2.15984494934298
- joint wheel_back: origin xyz=-0.1195 0 0.03 rpy=1.5708 0 -1.5708 -> xyz=-0.1195 0 0.03 rpy=1.5707963267949 0 -1.5707963267949
- joint wheel_left: axis -0.86603 0 -0.5 -> -0.866025403784436 0 -0.500000000000004; origin xyz=0.05975 0.10349 0.03 rpy=1.5708 0 -1.5708 -> xyz=0.0597500000000005 0.10349003575224 0.03 rpy=1.5707963267949 0 -1.5707963267949
- joint wheel_right: axis 0.86603 0 -0.5 -> 0.866025403784443 0 -0.499999999999992; origin xyz=0.059753 -0.10349 0.029998 rpy=1.5708 0 -1.5708 -> xyz=0.0597527016785317 -0.103488475937413 0.0299975068501592 rpy=1.5707963267949 0 -1.5707963267949
- joint wing_left: origin xyz=-0.171 0.338 -0.0087685 rpy=0 0 0 -> xyz=-0.171 0.337999997444124 -0.00876845650366815 rpy=0 0 0
- joint wing_right: origin xyz=0.171 0.338 -0.0087685 rpy=0 0 0 -> xyz=0.171 0.337999997444124 -0.00876845650366815 rpy=0 0 0

Commit message: adjusting ir sensors

File: sanbot_nano_urdf/urdf/sanbot_nano_urdf.urdf (robot description, URDF)
Before this commit: robot sanbot_nano_urdf, 29 links, 28 joints
Links:
- link base_link: geometry collision mesh filename=package://sanbot_nano_urdf/meshes/base_link.STL; visual mesh filename=package://sanbot_nano_urdf/textures/base.dae
- link body_link: geometry collision mesh filename=package://sanbot_nano_urdf/meshes/body_link.STL; visual mesh filename=package://sanbot_nano_urdf/textures/body.dae
- link camera_chin_link: geometry collision mesh filename=package://sanbot_nano_urdf/meshes/camera_chin_link.STL; visual mesh filename=package://sanbot_nano_urdf/textures/camera_chin.dae
- link camera_depth_link: geometry collision mesh filename=package://sanbot_nano_urdf/meshes/camera_depth_link.STL; visual mesh filename=package://sanbot_nano_urdf/textures/camera_depth.dae
- link camera_forehead_link: geometry collision mesh filename=package://sanbot_nano_urdf/meshes/camera_forehead_link.STL; visual mesh filename=package://sanbot_nano_urdf/textures/camera_forehead.dae
- link head_link: geometry collision mesh filename=package://sanbot_nano_urdf/meshes/head_link.STL; visual mesh filename=package://sanbot_nano_urdf/textures/head.dae
- link wing_left_link: geometry collision mesh filename=package://sanbot_nano_urdf/meshes/wing_left_link.STL; visual mesh filename=package://sanbot_nano_urdf/textures/wing_left.dae
- link wing_right_link: geometry collision mesh filename=package://sanbot_nano_urdf/meshes/wing_right_link.STL; visual mesh filename=package://sanbot_nano_urdf/textures/wing_right.dae
Joints:
- joint ir_1: origin xyz=0.145947826146462 0.0842630167133011 0.015 rpy=1.38875485932488 0.104144000510505 -1.05671160838547 -> xyz=0.145947826146462 0.0842630167133011 0.015 rpy=1.355 0.104144000510505 -1.05671160838547
- joint ir_2: origin xyz=0.145947826146462 -0.0842630167133002 0.015 rpy=1.38875485932488 -0.104144000510505 -2.08488104520432 -> xyz=0.145947826146462 -0.0842630167133002 0.015 rpy=1.355 -0.104144000510505 -2.08488104520432
